File: Eagle/Project/AdelinoR1.brd (EAGLE design)
At the start: 47 x 53.3 mm, 67 parts, among them J1 DC-044-A, J2 YELLOW-8P-2.54, J3 YELLOW-6P-2.54, J4 YELLOW-8P-2.54, J5 YELLOW-8P-2.54, J6 4P-2.0, J7 YELLOW-2X3P-2.54, J8 4P-2.0, Q1 NCE3407A, Q2 CJ2305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

Commit message: Fix USB connector D+/D- wiring.
Connections:
- net D+: now also R2.2; no longer R1.2
- net D-: now also R1.2; no longer R2.2
Routing:
- net D+: track 43.4 -> 42.7 mm
Changed lines of the file:
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@@
 <?xml version="1.0" encoding="utf-8"?>
 <!DOCTYPE eagle SYSTEM "eagle.dtd">
-<eagle version="9.2.1">
+<eagle version="9.2.2">
 <drawing>
 <settings>
@@
 <element name="C10" library="Seeed-Capacitor" package="C0402" value="22pf" x="34.036" y="45.9835" smashed="yes" rot="R90">
 <attribute name="MPN" value="CC0402JRNPO9BN220" x="34.036" y="45.9835" size="1.778" layer="27" rot="R90" display="off"/>
+<attribute name="NAME" x="32.766" y="45.7295" size="0.635" layer="33" ratio="10"/>
 <attribute name="NAME" x="33.528" y="45.8565" size="0.4064" layer="25" ratio="11"/>
-<attribute name="NAME" x="32.766" y="45.7295" size="0.635" layer="33" ratio="10"/>
 <attribute name="VALUE" x="32.766" y="44.396" size="0.635" layer="27" ratio="10"/>
 </element>
@@
 <element name="C9" library="Seeed-Capacitor" package="C0402" value="22pf" x="31.496" y="46.0195" smashed="yes" rot="R270">
 <attribute name="MPN" value="CC0402JRNPO9BN220" x="31.496" y="46.0195" size="1.778" layer="27" rot="R270" display="off"/>
+<attribute name="NAME" x="32.766" y="46.2735" size="0.635" layer="33" ratio="10" rot="R180"/>
 <attribute name="NAME" x="31.877" y="46.2735" size="0.4064" layer="25" ratio="11" rot="R180"/>
-<attribute name="NAME" x="32.766" y="46.2735" size="0.635" layer="33" ratio="10" rot="R180"/>
 <attribute name="VALUE" x="32.766" y="47.607" size="0.635" layer="27" ratio="10" rot="R180"/>
 </element>
@@
 <element name="J1" library="Seeed-Connector" package="DCJ3P-11.6X9.6X7.0MM" value="DC-044-A" x="0" y="9.906" smashed="yes" rot="R270">
 <attribute name="MPN" value="JACK-DC-044-A" x="0" y="9.906" size="1.778" layer="27" rot="R270" display="off"/>
+<attribute name="NAME" x="6.985" y="13.1445" size="1.27" layer="33" ratio="10" rot="R270"/>
 <attribute name="NAME" x="3.3655" y="11.811" size="0.889" layer="25" ratio="11"/>
-<attribute name="NAME" x="6.985" y="13.1445" size="1.27" layer="33" ratio="10" rot="R270"/>
 <attribute name="VALUE" x="4.3815" y="3.556" size="0.889" layer="27" ratio="11"/>
 </element>
 <element name="J3" library="Seeed-Connector" package="H6-2.54" value="YELLOW-6P-2.54" x="35.56" y="2.54" smashed="yes" rot="R90">
 <attribute name="MPN" value="F185-1106A1BSYA3" x="35.56" y="2.54" size="1.778" layer="27" rot="R90" display="off"/>
+<attribute name="NAME" x="38.1" y="3.175" size="0.635" layer="33" ratio="10" rot="R180"/>
 <attribute name="NAME" x="36.195" y="2.921" size="0.889" layer="25" ratio="11" rot="R180"/>
-<attribute name="NAME" x="38.1" y="3.175" size="0.635" layer="33" ratio="10" rot="R180"/>
 <attribute name="VALUE" x="37.465" y="5.08" size="0.889" layer="27" ratio="11" rot="R180"/>
 </element>
 <element name="J2" library="Seeed-Connector" package="H8-2.54" value="YELLOW-8P-2.54" x="15.24" y="2.54" smashed="yes" rot="R90">
 <attribute name="MPN" value="F185-1108A1BSYC1" x="15.24" y="2.54" size="1.778" layer="27" rot="R90" display="off"/>
+<attribute name="NAME" x="15.875" y="2.54" size="0.3048" layer="33" ratio="10" rot="R180"/>
 <attribute name="NAME" x="15.748" y="2.921" size="0.889" layer="25" ratio="11" rot="R180"/>
-<attribute name="NAME" x="15.875" y="2.54" size="0.3048" layer="33" ratio="10" rot="R180"/>
 <attribute name="VALUE" x="16.51" y="5.08" size="0.889" layer="27" ratio="11" rot="R180"/>
 </element>
 <element name="J5" library="Seeed-Connector" package="H8-2.54" value="YELLOW-8P-2.54" x="33.02" y="50.8" smashed="yes" rot="R270">
 <attribute name="MPN" value="F185-1108A1BSYC1" x="33.02" y="50.8" size="1.778" layer="27" rot="R270" display="off"/>
+<attribute name="NAME" x="32.385" y="50.8" size="0.3048" layer="33" ratio="10"/>
 <attribute name="NAME" x="32.512" y="50.419" size="0.889" layer="25" ratio="11"/>
-<attribute name="NAME" x="32.385" y="50.8" size="0.3048" layer="33" ratio="10"/>
 <attribute name="VALUE" x="31.75" y="48.26" size="0.889" layer="27" ratio="11"/>
 </element>
 <element name="J4" library="Seeed-Connector" package="H8-2.54" value="YELLOW-8P-2.54" x="11.43" y="50.8" smashed="yes" rot="R270">
 <attribute name="MPN" value="F185-1108A1BSYC1" x="11.43" y="50.8" size="1.778" layer="27" rot="R270" display="off"/>
+<attribute name="NAME" x="10.795" y="50.8" size="0.3048" layer="33" ratio="10"/>
 <attribute name="NAME" x="10.668" y="50.419" size="0.889" layer="25" ratio="11"/>
-<attribute name="NAME" x="10.795" y="50.8" size="0.3048" layer="33" ratio="10"/>
 <attribute name="VALUE" x="10.16" y="48.26" size="0.889" layer="27" ratio="11"/>
 </element>
@@
 </signal>
 <signal name="D+">
-<contactref element="R1" pad="2"/>
 <contactref element="U4" pad="4"/>
 <via x="10.6552375" y="36.83" extent="1-16" drill="0.6096"/>
@@
 <wire x1="29.8196" y1="34.671" x2="29.4386" y2="34.29" width="0.254" layer="1"/>
 <wire x1="38.312" y1="33.198" x2="37.3886" y2="33.198" width="0.254" layer="1"/>
-<wire x1="11.0035" y1="37.8915" x2="11.0035" y2="37.1782625" width="0.254" layer="1"/>
 <wire x1="11.0035" y1="37.1782625" x2="10.6552375" y2="36.83" width="0.254" layer="1"/>
 <wire x1="28.618575" y1="34.29" x2="22.395575" y2="28.067" width="0.254" layer="16"/>
@@
 <wire x1="9.144" y1="34.036" x2="8.89" y2="33.782" width="0.254" layer="16"/>
 <wire x1="9.652" y1="34.036" x2="9.144" y2="34.036" width="0.254" layer="16"/>
+<contactref element="R2" pad="2"/>
+<wire x1="9.906" y1="34.544" x2="11.0035" y2="35.0615" width="0" layer="19" extent="1-16"/>
 </signal>
 <signal name="D-">
-<contactref element="R2" pad="2"/>
 <contactref element="U4" pad="3"/>
 <via x="9.398" y="36.5815" extent="1-16" drill="0.6096"/>
@@
 <wire x1="10.1655" y1="35.814" x2="10.414" y2="35.814" width="0.254" layer="1"/>
 <wire x1="10.414" y1="35.814" x2="11.0035" y2="35.2245" width="0.254" layer="1"/>
-<wire x1="11.0035" y1="35.2245" x2="11.0035" y2="35.0615" width="0.254" layer="1"/>
+<contactref element="R1" pad="2"/>
+<wire x1="9.398" y1="36.5815" x2="11.0035" y2="37.8915" width="0" layer="19" extent="1-1"/>
 </signal>
 <signal name="UGND">
