File: Eagle/Project/AdelinoR2.brd (EAGLE design)
At the start: 47 x 53.3 mm, 76 parts, among them J1 DC-044-A, J2 YELLOW-8P-2.54, J3 YELLOW-6P-2.54, J4 YELLOW-8P-2.54, J5 YELLOW-8P-2.54, J6 4P-2.0, J7 YELLOW-2X3P-2.54, J8 4P-2.0, Q1 NCE3407A, Q2 CJ2305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

Commit message: Wip.
Parts:
- removed D4, D5: YEL-0603, Seeed-LED:LED-0603
- removed D6: GRE-0603, Seeed-LED:LED-0603
- removed U5: 74VHC125MTCX-TSSOP14, Seeed-IC:TSSOP14-0.65-5X4.4MM
- added R23, R24, R25, R26: 1K, Seeed-Resistor:R0402
- added R27: 470R, Seeed-Resistor:R0402
- added R28: 10K, Seeed-Resistor:R0402
- added R29: 0R, Seeed-Resistor:R0402
- R10, R5: value 10K 1/16W -> 10K
- R11, R12: value 1K -> 10K; device Seeed-Resistor:RA1206-8 -> Seeed-Resistor:R0402
- moved R11 148.1 mm to (-101.9, -29.7)
- moved R12 146.0 mm to (-105.9, -29.7)
Connections:
- removed net CH_EN: U3.3, U5.11
- removed net D13_LED: R11.6, U5.8
- removed net GPIO15_PD: R12.4, U3.16
- removed net GPIO2: R11.5
- removed net GPIO2_PU: R12.2, U3.17
- removed net HSPI_CLK: U3.5
- removed net HSPI_MISO: U3.6
- removed net HSPI_MOSI: U3.7
- removed net N$11: D6.-, R11.1
- removed net N$16: R12.3
- removed net N$8: D5.-, R11.2
- removed net RESET_AT: U3.4, U5.1, U5.2
- removed net RST_PU: R12.1, U3.1
- new net GPIO2_LED: D8.-, R28.2, U3.17
- new net N$12: R23.2, U3.6
- new net N$14: R24.2, U3.7
- new net N$19: R25.2, U3.5
- new net N$20: R12.2, R26.2, U3.16
- new net N$22: R10.2, U3.1
- net +3V3: now also R10.1, R11.2, R27.1, R28.1, R5.1; no longer D8.+, R12.6, R12.7, R12.8
- net +5V: no longer D4.+, D5.+, D6.+, R10.2, R5.2, U5.14
- net ACT_LED: no longer R11.7
- net AT_MISO: now also R23.1
- net AT_MOSI: now also R24.1; no longer R10.1, U5.5
- net AT_SCK: now also R25.1
- net AT_SS: now also R26.1
- net BOOT_MODE: now also R11.1; no longer U5.6
- net ESP_EN: now also R5.2, U3.3; no longer R5.1, U5.12
- net GND: now also R12.1; no longer R11.8, R12.5, U5.10, U5.13, U5.4, U5.7
- net N$5: now also R29.2, U3.4; no longer D8.-, R11.4
- net N$6: now also D8.+, R27.2; no longer D4.-, R11.3
- net PIN_D0: now also J8.1
- net PIN_D1: now also J8.2
- net PIN_D10: no longer J8.1
- net PIN_D13: no longer U5.9
- net PIN_D2: now also U3.19; no longer U3.20
- net PIN_D3: now also U3.20; no longer U3.19
- net PIN_D9: no longer J8.2
- net RESET: now also R29.1; no longer U5.3
