File: Eagle/Project/AdelinoR2.sch (EAGLE design)
At the start: 79 parts, among them J1 DC-044-A, J2 YELLOW-8P-2.54, J3 YELLOW-6P-2.54, J4 YELLOW-8P-2.54, J5 YELLOW-8P-2.54, J6 4P-2.0, J7 YELLOW-2X3P-2.54, J8 4P-2.0, Q1 NCE3407A, Q2 CJ2305, SW1 TS-1101F, U1 MP1496DJ-SOT23-8, U2 CJT1117-3.3-SOT223, U3 ESP-12F / OPL: 317060163 / SM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, U4 ATMEGA32U4-MUR-QFN44, U6 ATMEGA32U4-TQFP44, X1 306010049_XTAL_16MHZ-3225_4P

Commit message: Routing wip.
Parts:
- removed D10: YEL-0603, Seeed-LED:SMD-LED-CLEAR-YELLOW(0603)
- added D4: GRE-0603, Seeed-LED:SMD-LED-CLEAR-GREEN(0603)
- C1, C19, C4, C8: value 10uf -> 100nf; device Seeed-Capacitor:CERAMIC-10UF-25V-10%-X5R(0805) -> Seeed-Capacitor:CERAMIC-100NF-25V-10%-X7R(0402)
- C10, C9: value 22pf -> 10uf; device Seeed-Capacitor:CERAMIC-22PF-50V-5%-NPO(0402) -> Seeed-Capacitor:CERAMIC-10UF-25V-10%-X5R(0805)
- C12, C13: value 100nf -> 22pf; device Seeed-Capacitor:CERAMIC-100NF-25V-10%-X7R(0402) -> Seeed-Capacitor:CERAMIC-22PF-50V-5%-NPO(0402)
- C16: value 1uf -> 100nf; device Seeed-Capacitor:CERAMIC-1UF-25V-10%-X7R(0805) -> Seeed-Capacitor:CERAMIC-100NF-25V-10%-X7R(0402)
- C2, C6: value 100nf -> 10uf; device Seeed-Capacitor:CERAMIC-100NF-25V-10%-X7R(0402) -> Seeed-Capacitor:CERAMIC-10UF-25V-10%-X5R(0805)
- C20: value 10uf -> 1uf; device Seeed-Capacitor:CERAMIC-10UF-25V-10%-X5R(0805) -> Seeed-Capacitor:CERAMIC-1UF-25V-10%-X7R(0805)
- C3: value 22NF 50V -> 10uf; device Seeed-Capacitor:CERAMIC-22NF-50V-10%-X7R(0402) -> Seeed-Capacitor:CERAMIC-10UF-25V-10%-X5R(0805)
- C7: value 100nf -> 22NF 50V; device Seeed-Capacitor:CERAMIC-100NF-25V-10%-X7R(0402) -> Seeed-Capacitor:CERAMIC-22NF-50V-10%-X7R(0402)
- D3: value GRE-0603 -> 20V-500MA; device Seeed-LED:SMD-LED-CLEAR-GREEN(0603) -> Seeed-Diode:SMD-DIODE-SCHOTTKY-20V-500MA(SOD-123)P; LABEL PWR -> (none)
- D7: value 20V-500MA -> YEL-0603; device Seeed-Diode:SMD-DIODE-SCHOTTKY-20V-500MA(SOD-123)P -> Seeed-LED:SMD-LED-CLEAR-YELLOW(0603); LABEL (none) -> D13
- R1: value 22R -> 100K; device Seeed-Resistor:SMD-RES-22R-1%-1/16W(0402) -> Seeed-Resistor:SMD-RES-100K-1%-1/16W(0402)
- R10: value 10K -> 100K; device Seeed-Resistor:SMD-RES-10K-1%-1/16W(0402) -> Seeed-Resistor:SMD-RES-100K-1%-1/16W(0402)
- R12: value 10K -> 1M; device Seeed-Resistor:SMD-RES-10K-1%-1/16W(0402) -> Seeed-Resistor:SMD-RES-1M-1%-1/16W(0402)
- R13: value 2K7 / 1% -> 10K; device Seeed-Resistor:SMD-RES-2.7K-1%-1/10W(0603) -> Seeed-Resistor:SMD-RES-10K-1%-1/16W(0402); R 2K7 / 1% -> (none)
- R14, R23: value 1K -> 10K; device Seeed-Resistor:SMD-RES-1K-5%-1/16W(0402) -> Seeed-Resistor:SMD-RES-10K-1%-1/16W(0402)
- R15: value 3K / 1% -> 1K; device Seeed-Resistor:SMD-RES-510R-1%-1/10W(0603) -> Seeed-Resistor:SMD-RES-1K-5%-1/16W(0402); R 510R / 1% -> (none)
- R17: value 100K -> 1K; device Seeed-Resistor:SMD-RES-100K-1%-1/16W(0402) -> Seeed-Resistor:SMD-RES-1K-5%-1/16W(0402)
- R18: value 3.3K -> 1K; device Seeed-Resistor:SMD-RES-3.3K-5%-1/16W(0402) -> Seeed-Resistor:SMD-RES-1K-5%-1/16W(0402)
- R19: value 100K -> 0R; device Seeed-Resistor:SMD-RES-100K-1%-1/16W(0402) -> Seeed-Resistor:SMD-RES-0R-5%-1/16W(0402)
- R27: value 470R -> 1K; device Seeed-Resistor:SMD-RES-470R-5%-1/16W(0402) -> Seeed-Resistor:SMD-RES-1K-5%-1/16W(0402)
- R28: value 10K -> 470R; device Seeed-Resistor:SMD-RES-10K-1%-1/16W(0402) -> Seeed-Resistor:SMD-RES-470R-5%-1/16W(0402)
- R29: value 0R -> 10K; device Seeed-Resistor:SMD-RES-0R-5%-1/16W(0402) -> Seeed-Resistor:SMD-RES-10K-1%-1/16W(0402)
- R3: value 100K -> 22R; device Seeed-Resistor:SMD-RES-100K-1%-1/16W(0402) -> Seeed-Resistor:SMD-RES-22R-1%-1/16W(0402)
- R4: value 1M -> 10R 1/16W; device Seeed-Resistor:SMD-RES-1M-1%-1/16W(0402) -> Seeed-Resistor:SMD-RES-10R-1%-1/16W(0402)
- R5: value 10K -> 3.3K; device Seeed-Resistor:SMD-RES-10K-1%-1/16W(0402) -> Seeed-Resistor:SMD-RES-3.3K-5%-1/16W(0402)
- R6: value 10R 1/16W -> 3K / 1%; device Seeed-Resistor:SMD-RES-10R-1%-1/16W(0402) -> Seeed-Resistor:SMD-RES-510R-1%-1/10W(0603); R (none) -> 510R / 1%
- R7: value 100K -> 2K7 / 1%; device Seeed-Resistor:SMD-RES-100K-1%-1/16W(0402) -> Seeed-Resistor:SMD-RES-2.7K-1%-1/10W(0603); R (none) -> 2K7 / 1%
- R8, R9: value 1K -> 100K; device Seeed-Resistor:SMD-RES-1K-5%-1/16W(0402) -> Seeed-Resistor:SMD-RES-100K-1%-1/16W(0402)
- U1: value MP1496DJ-SOT23-8 -> CJT1117-3.3-SOT223; device Seeed-IC:PMIC-MP1496DJ(SOT23-8) -> Seeed-IC:PMIC-CJT1117-3.3(SOT223)
- U2: value CJT1117-3.3-SOT223 -> MP1496DJ-SOT23-8; device Seeed-IC:PMIC-CJT1117-3.3(SOT223) -> Seeed-IC:PMIC-MP1496DJ(SOT23-8)
- renumbered D11 to D6, D9 to D5, U6 to U5
Connections:
- removed net N$10: D10.+, R16.2
- removed net N$4: D3.+, R21.2
- removed net N$6: D8.+, R27.2
- removed net N$7: D5.+, D6.+, R22.2
- new net _ACT: D5.+, D6.+, R25.2
- new net _D13: D7.+, R26.2
- new net _ESP: D8.+, R28.2
- new net _PWR: D4.+, R24.2
- net +3V3: now also C4.2, C6.2, R13.1, R14.1, R23.2, R29.1, U1.OUT; no longer C7.2, C8.2, R10.1, R11.2, R27.1, R5.1, U2.OUT
- net +5V: now also C1.2, C10.2, C15.1, C16.1, C17.1, C18.1, C9.2, D3.-, R10.2, R24.1, R7.2, R8.1, R9.1, U1.IN; no longer C11.1, C12.1, C13.1, C14.1, C19.2, C20.2, C6.2, D7.-, R13.2, R17.1, R19.2, R21.1, R3.1, U2.IN
- net ACT_LED: now also R25.1; no longer R22.1
- net AT_MISO: now also R15.1; no longer R23.1
- net AT_MOSI: now also R16.1; no longer R24.1
- net AT_SCK: now also R17.1; no longer R25.1
- net AT_SS: now also R18.1; no longer R26.1
- net BOOT_MODE: now also R23.1, R27.2; no longer R11.1, R14.2
- net D+: now also R3.2; no longer R2.2
- net D-: now also R2.2; no longer R1.2
- net ESP_EN: now also R14.2; no longer R5.2
- net GND: now also C12.1, C13.1, C16.2, C17.2, C19.2, C5.1, D4.-, D7.-, R20.1, R6.1, SW1.1; no longer C11.2, C12.2, C13.2, C19.1, C20.1, C8.1, D10.-, D3.-, R12.1, R15.1, SW1.2
- net GPIO2_LED: now also R29.2; no longer R28.2
- net N$1: now also R2.1; no longer R1.1
- net N$12: now also R15.2; no longer R23.2
- net N$13: now also C14.1, R11.2; no longer C18.1, R20.2
- net N$14: now also R16.2; no longer R24.2
- net N$15: now also C8.2, R4.2; no longer C5.2, R6.2
- net N$17: now also R21.1; no longer R8.1
- net N$18: now also R22.1; no longer R9.1
- net N$19: now also R17.2; no longer R25.2
- net N$2: now also R3.1; no longer R2.1
- net N$20: now also R18.2, R20.2; no longer R12.2, R26.2
- net N$22: now also R13.2; no longer R10.2
- net N$23: now also R5.2, R6.2, R7.1; no longer R13.1, R15.2, R18.2
- net N$3: now also R8.2; no longer R3.2
- net N$5: now also R19.2; no longer R29.2
- net PIN_AREF: now also C19.1; no longer C15.1
- net PIN_D0: now also R21.2; no longer R8.2
- net PIN_D1: now also R22.2; no longer R9.2
- net PIN_D13: now also R26.1, R27.1; no longer R14.1, R16.1
- net RESET: now also C11.1, D3.+, R10.1, R11.1; no longer C17.1, D7.+, R20.1, R29.1
- net RSTAT: now also C11.2, R9.2, SW1.2; no longer C17.2, R17.2, SW1.1
- net SW_BS: now also R4.1, U2.BS; no longer R6.1, U1.BS
- net SW_EN: now also R1.1, U2.EN/SYNC; no longer R7.1, U1.EN/SYNC
- net SW_FB: now also R5.1, U2.FB; no longer R18.1, U1.FB
- net SW_SS: now also C7.2, U2.SS; no longer C3.2, U1.SS
- net SW_VCAP: now also C5.2, U2.VCC; no longer C2.2, U1.VCC
- net SW_VCC_IN: now also C2.2, C3.2, R1.2, U2.IN; no longer C1.2, C4.2, R7.2, U1.IN
- net SW_VCC_OUT: now also C8.1, U2.SW; no longer C5.1, U1.SW
- net UCAP: now also C20.2; no longer C16.2
- net UGND: now also C20.1; no longer C16.1
- net XTAL1: now also C12.2, R12.2; no longer C9.2, R4.2
- net XTAL2: now also C13.2, R12.1; no longer C10.2, R4.1
Other:
- moved on the sheet: C1, C10, C11, C12, C13, C14, C15, C16, C17, C18, C19, C2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
