File: Eagle/Project/AdelinoX2/AdelinoR2.sch (EAGLE design)
At the start: 80 parts, among them J1 DC-044-A, J2 YELLOW-8P-2.54, J3 YELLOW-6P-2.54, J4 YELLOW-8P-2.54, J5 YELLOW-8P-2.54, J6 4P-2.0, J7 YELLOW-2X3P-2.54, J8 4P-2.0, Q1 NCE3407A, Q2 CJ2305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

Commit message: Preparing pcb for Revision A.
Parts:
- D1: value SMBJ15CA-13-F -> TVS-DIODE-SZOPL-SMBJ15CA-13-F; device Adelino-Misc:SMBJ15CA-13-F -> Adelino-Misc:TVS-DIODE-SZOPL-SMBJ15CA-13-F
Changed lines of the file:
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@@
 </variantdefs>
 <classes>
-<class number="0" name="default" width="0.254" drill="0.6096">
+<class number="0" name="default" width="0.2032" drill="0.2032">
 <clearance class="0" value="0.254"/>
 </class>
@@
 <part name="P+6" library="supply1" library_urn="urn:adsk.eagle:library:371" deviceset="+5V" device=""/>
 <part name="C21" library="Seeed-Capacitor" deviceset="CERAMIC-100NF-25V-10%-X7R(0402)" device="" value="100nf"/>
-<part name="D1" library="Adelino-Misc" deviceset="SMBJ15CA-13-F" device=""/>
+<part name="D1" library="Adelino-Misc" deviceset="TVS-DIODE-SZOPL-SMBJ15CA-13-F" device=""/>
 </parts>
 <sheets>
